Commit message: Improve sensor runtime isolation and lidar filtering

File: modules/robot_description/ranger/urdf/ranger_mini_v3.urdf (robot description, URDF)
Before this commit: robot ranger_mini_v3, 32 links, 31 joints
Links:
- added link rslidar
Joints:
- added joint rslidar_frame_joint: type fixed, parent lidar_link, child rslidar, origin xyz=0 0 0 rpy=0 0 0, axis 0 0 0
