Commit message: calibration

File: modules/robot_description/ranger/urdf/ranger_mini_v3.urdf (robot description, URDF)
Before this commit: robot ranger_mini_v3, 33 links, 32 joints
Joints:
- joint lifting_joint: limit lower=-0.6 upper=0.0 effort=100 velocity=10.0 -> lower=0.0 upper=0.75 effort=100 velocity=10.0
